File: class2.2/load_box.kicad_pcb (KiCad board)
At the start: 2 copper layers, 16 parts, among them J1 CONN_01X02, J2 CONN_01X02, U1 STM32L152C6TxA, Y1 Crystal_GND24

Commit message: checkpoint some analog
Parts:
- removed L1: Ferrite_Bead, Inductors_SMD:L_0603
- removed Y1: Crystal_GND24, Crystals:Crystal_SMD_EuroQuartz_MJ-4pin_5.0x3.2mm
- added D1: D, Diodes_SMD:D_SOD-123, F.Cu at (134.0, 107.3)
- added D2: D, Diodes_SMD:D_SOD-123, F.Cu at (134.0, 112.4)
- added D3: D, Diodes_SMD:D_SOD-123, F.Cu at (123.2, 63.5)
- added J3: Screw_Terminal_1x02, Connectors_Terminal_Blocks:TerminalBlock_Pheonix_MKDS1.5-2pol, F.Cu at (199.4, 77.5)
- added Q1: Q_NMOS_GDS, TO_SOT_Packages_SMD:SOT-23, F.Cu at (123.8, 67.3)
- added Q2: Q_NMOS_GDS, TO_SOT_Packages_THT:TO-220_Vertical, F.Cu at (181.0, 64.1)
- added Q3: Q_NMOS_GDS, TO_SOT_Packages_THT:TO-220_Vertical, F.Cu at (135.9, 64.1)
- added R10: R, Resistors_SMD:R_0603, F.Cu at (124.5, 72.4)
- added R11: 100R, Resistors_SMD:R_0603, F.Cu at (176.5, 67.3)
- added R12: R, Resistors_THT:R_Axial_DIN0516_L15.5mm_D5.0mm_P20.32mm_Horizontal, F.Cu at (191.1, 72.4)
- added R13: R, Resistors_THT:R_Axial_DIN0516_L15.5mm_D5.0mm_P20.32mm_Horizontal, F.Cu at (178.4, 72.4)
- added R14: R, Resistors_THT:R_Axial_DIN0516_L15.5mm_D5.0mm_P20.32mm_Horizontal, F.Cu at (184.8, 72.4)
- added R15: R, Resistors_THT:R_Axial_DIN0516_L15.5mm_D5.0mm_P20.32mm_Horizontal, F.Cu at (172.1, 72.4)
- added R16: 100R, Resistors_SMD:R_0603, F.Cu at (146.7, 67.9)
- added R19: R, Resistors_SMD:R_0603, F.Cu at (187.3, 97.2)
- added R23: R, Resistors_SMD:R_0603, F.Cu at (191.8, 96.5)
- added R24: R, Resistors_SMD:R_0603, F.Cu at (191.8, 97.2)
- added R25: R, Resistors_SMD:R_0603, F.Cu at (193.0, 104.8)
- added R26: R, Resistors_SMD:R_0603, F.Cu at (192.4, 101.0)
- added R3: R, Resistors_SMD:R_0603, F.Cu at (134.0, 97.8)
- added R4: R, Resistors_SMD:R_0603, F.Cu at (150.5, 103.5)
- added R5: R, Resistors_SMD:R_0603, F.Cu at (141.6, 104.1)
- added R6: R, Resistors_SMD:R_0603, F.Cu at (160.0, 97.8)
- added R7: R, Resistors_SMD:R_0603, F.Cu at (146.1, 98.4)
- added R8: R, Resistors_SMD:R_0603, F.Cu at (153.0, 100.3)
- added R9: R, Resistors_SMD:R_0603, F.Cu at (161.3, 89.5)
- added RV1: POT_TRIM, Potentiometers:Potentiometer_Trimmer_Bourns_3214G, F.Cu at (160.0, 66.0)
- added TH1: Thermistor_NTC, Connectors_JST:JST_XH_B02B-XH-A_02x2.50mm_Straight, F.Cu at (166.4, 65.4)
- added TP1: TEST, Measurement_Points:Test_Point, F.Cu at (160.0, 95.9)
- added TP2: TEST, Measurement_Points:Test_Point, F.Cu at (145.4, 100.3)
- added TP3: TEST, Measurement_Points:Test_Point, F.Cu at (152.4, 99.1)
- added TP4: TEST, Measurement_Points:Test_Point, F.Cu at (146.1, 106.7)
- added TP5: TEST, Measurement_Points:Test_Point, F.Cu at (173.4, 64.1)
- added TP6: TEST, Measurement_Points:Test_Point, F.Cu at (164.5, 98.4)
- added TP7: TEST, Measurement_Points:Test_Point, F.Cu at (167.6, 96.5)
- added TP8: TEST, Measurement_Points:Test_Point, F.Cu at (146.1, 64.1)
- added U2: INA128, Housings_SOIC:SOIC-8_3.9x4.9mm_Pitch1.27mm, F.Cu at (187.3, 102.2)
- C7, C8: value C -> 0.1
- J1: footprint Buttons_Switches_THT:SW_PUSH_6mm_h9.5mm -> Connectors_JST:JST_XH_B02B-XH-A_02x2.50mm_Straight
- J2: value CONN_01X02 -> Screw_Terminal_1x02; footprint Buttons_Switches_THT:SW_PUSH_6mm_h9.5mm -> Connectors_Terminal_Blocks:TerminalBlock_Pheonix_MKDS1.5-2pol
- U1: value STM32L152C6TxA -> LM324; footprint Housings_QFP:LQFP-48_7x7mm_Pitch0.5mm -> Housings_SOIC:SOIC-14_3.9x8.7mm_Pitch1.27mm
- moved J2 91.6 mm to (199.4, 99.1), turned to 270 degrees
- moved C5 56.3 mm to (167.0, 135.3)
- moved C1 30.7 mm to (179.1, 102.2)
- moved C2 27.5 mm to (139.6, 131.0)
- moved C3 27.5 mm to (139.6, 131.0)
- moved C4 27.5 mm to (139.6, 131.0)
- moved C6 27.5 mm to (139.6, 131.0)
- moved C7 27.5 mm to (139.6, 131.0)
- moved C8 27.5 mm to (139.6, 131.0)
- moved C9 27.5 mm to (139.6, 131.0)
- moved R1 27.5 mm to (139.6, 131.0)
- moved R2 27.5 mm to (139.6, 131.0)
- moved U1 21.3 mm to (154.9, 81.9)
- moved J1 12.1 mm to (113.7, 69.2), turned to 90 degrees
Connections:
- C1 pad 1: Net-(C1-Pad1) -> GND
- C1 pad 2: GND -> (no net)
- C2 pad 1: Net-(C2-Pad1) -> GND
- C2 pad 2: GND -> +3V3
- C3 pad 1: Net-(C3-Pad1) -> GND
- C3 pad 2: Net-(C3-Pad2) -> +3V3
- C4 pad 1: RSTB -> (no net)
- C5 pad 1: +5V -> +3V3
- C6 pad 1: +5V -> (no net)
- C7 pad 1: +5V -> +12V
- C8 pad 1: +5V -> +12V
- J1 pad 1: GND -> +12V
- J1 pad 2: RSTB -> Net-(D3-Pad2)
- J2 pad 1: GND -> Net-(J2-Pad1)
- J2 pad 2: USERB -> Net-(J2-Pad2)
- R1 pad 1: +5V -> (no net)
- U1 pad 1: Net-(U1-Pad1) -> Net-(R8-Pad1)
- U1 pad 11: Net-(U1-Pad11) -> GND
- U1 pad 12: Net-(U1-Pad12) -> (no net)
- U1 pad 13: Net-(U1-Pad13) -> Net-(R8-Pad1)
- U1 pad 2: USERB -> Net-(R8-Pad2)
- U1 pad 3: Net-(C1-Pad1) -> Net-(R6-Pad2)
- U1 pad 4: Net-(C2-Pad1) -> +12V
- U1 pad 6: Net-(U1-Pad6) -> /load_box_sink/MEASURED_VREF
- U1 pad 7: RSTB -> /load_box_sink/MEASURED_VREF
- U1 pad 8: AVDD -> Net-(R10-Pad2)
- U1 pad 9: GND -> Net-(R5-Pad2)

Commit message: Further layout.
Parts:
- added C10: 0.1u, Capacitors_SMD:C_0603, F.Cu at (122.6, 119.4)
- added C11: 10u, Capacitors_SMD:C_1206, F.Cu at (130.2, 106.0)
- added C12: 0.1u, Capacitors_SMD:C_0603, F.Cu at (126.4, 126.4)
- added C13: 10u, Capacitors_SMD:C_1206, F.Cu at (135.9, 106.0)
- added C18: 0.1, Capacitors_SMD:C_0603, F.Cu at (178.1, 153.6)
- added C19: 0.1, Capacitors_SMD:C_0603, F.Cu at (207.9, 136.5)
- added J6: CONN_01X02, Connectors_JST:JST_XH_B02B-XH-A_02x2.50mm_Straight, F.Cu at (117.5, 67.3)
- added L1: 10uH, Inductors_SMD:L_Wuerth_MAPI-2510, F.Cu at (127.0, 114.9)
- added R18: R, Resistors_SMD:R_0603, F.Cu at (211.2, 137.1)
- added R20: R, Resistors_SMD:R_0603, F.Cu at (196.6, 155.7)
- added SW1: SW_SPST, Buttons_Switches_THT:SW_SPDT, F.Cu at (121.3, 104.8)
- added U3: LD1117S50TR, TO_SOT_Packages_SMD:SOT-223, F.Cu at (130.2, 89.5)
- added U4: STM32L152RCTx, Housings_QFP:LQFP-64_10x10mm_Pitch0.5mm, F.Cu at (145.4, 116.2)
- added U5: AP3012, TO_SOT_Packages_SMD:SOT-23-5, F.Cu at (130.2, 109.9)
- added U6: LD1117S33TR, TO_SOT_Packages_SMD:SOT-223, F.Cu at (130.2, 99.1)
- C7, C8: value 0.1 -> 1u
- J1: value CONN_01X02 -> BARREL_JACK; footprint Connectors_JST:JST_XH_B02B-XH-A_02x2.50mm_Straight -> Connectors:BARREL_JACK
- R5: value R -> 90.9k
- R6: value R -> 8.45k
- moved R16 111.2 mm to (134.5, 178.5)
- moved R10 108.8 mm to (203.2, 147.5)
- moved R19 92.6 mm to (134.9, 173.5)
- moved TP8 90.9 mm to (161.5, 153.7)
- moved TP5 87.9 mm to (172.4, 152.0)
- moved R9 87.1 mm to (138.0, 173.5)
- moved R25 86.3 mm to (134.9, 168.5)
- moved R11 81.3 mm to (208.4, 142.1)
- moved C1 79.0 mm to (147.5, 174.7)
- moved R3 78.4 mm to (154.4, 173.5)
- moved R4 70.3 mm to (157.3, 173.5)
- moved R7 69.8 mm to (200.3, 142.5)
- moved R8 69.8 mm to (138.0, 168.5)
- moved D1 62.7 mm to (145.2, 169.0)
- moved TP3 62.6 mm to (202.2, 137.0)
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Connections:
- net /load_box_sink/MEASURED_VREF renamed /load_box_mcu/MEASURED_VREF
- C7 pad 1: +12V -> +BATT
- C8 pad 1: +12V -> /load_box_display/+13V
- J1 pad 1: +12V -> Net-(J1-Pad1)
- J1 pad 2: Net-(D3-Pad2) -> GND
- R1 pad 1: (no net) -> +5V
- R5 pad 1: +12V -> /load_box_display/+13V
- R6 pad 1: /load_box_sink/CHOSEN_VREF -> Net-(R5-Pad2)
- R6 pad 2: Net-(R6-Pad2) -> GND
- R7 pad 1: Net-(R6-Pad2) -> Net-(R20-Pad2)
- TH1 pad 1: Net-(R5-Pad2) -> Net-(R18-Pad2)
- TP1 pad 1: /load_box_sink/CHOSEN_VREF -> /load_box_mcu/CHOSEN_VREF
- TP2 pad 1: Net-(R6-Pad2) -> Net-(R20-Pad2)
- U1 pad 3: Net-(R6-Pad2) -> Net-(R20-Pad2)
- U1 pad 9: Net-(R5-Pad2) -> Net-(R18-Pad2)

Commit message: Checkpoint with NHD, 3.3v, and layout
Parts:
- removed C13: 10u, Capacitors_SMD:C_1206
- removed J6: CONN_01X02, Connectors_JST:JST_XH_B02B-XH-A_02x2.50mm_Straight
- removed L1: 10uH, Inductors_SMD:L_Wuerth_MAPI-2510
- removed Q1: Q_NMOS_GDS, TO_SOT_Packages_SMD:SOT-23
- removed R18, R19, R20, R23, R24, R25, R26: R, Resistors_SMD:R_0603
- removed TH1: Thermistor_NTC, Connectors_JST:JST_XH_B02B-XH-A_02x2.50mm_Straight
- removed TP1, TP2, TP3, TP5, TP6, TP7, TP8: TEST, Measurement_Points:Test_Point
- removed U2: INA128, Housings_SOIC:SOIC-8_3.9x4.9mm_Pitch1.27mm
- removed U3: LD1117S50TR, TO_SOT_Packages_SMD:SOT-223
- removed U5: AP3012, TO_SOT_Packages_SMD:SOT-23-5
- added 1M1: R, Resistors_SMD:R_0603, F.Cu at (118.1, 119.4)
- added C14: C, Capacitors_SMD:C_0603, F.Cu at (153.0, 113.7)
- added C15: C, Capacitors_SMD:C_0603, F.Cu at (146.1, 106.7)
- added C16: C, Capacitors_SMD:C_0603, F.Cu at (131.4, 113.0)
- added C17: C, Capacitors_SMD:C_0603, F.Cu at (137.8, 124.5)
- added J4: CONN_02X10, nhd:NHD-1.69, F.Cu at (149.2, 78.7)
- added J5: Screw_Terminal_1x02, Connectors_Terminal_Blocks:TerminalBlock_Pheonix_MKDS1.5-2pol, F.Cu at (168.3, 113.0)
- added J7: USB_B, Connectors:USB_B, F.Cu at (121.9, 110.5)
- added J8: CONN_01X03, Socket_Strips:Socket_Strip_Straight_1x03_Pitch2.54mm, F.Cu at (138.4, 97.8)
- added L2: Ferrite_Bead, Inductors_SMD:L_0603, F.Cu at (153.0, 118.7)
- added RV2: POT, Potentiometers:Potentiometer_Alps_RK09K_Horizontal, F.Cu at (154.9, 131.4)
- added SW2: SW_Push, Buttons_Switches_THT:SW_Tactile_SKHH_Angled, F.Cu at (113.7, 80.0)
- added SW3: SW_Push, Buttons_Switches_THT:SW_Tactile_SKHH_Angled, F.Cu at (113.7, 92.1)
- added SW4: SW_Push, Pin_Headers:Pin_Header_Straight_1x02_Pitch2.54mm, F.Cu at (170.8, 139.1)
- added Y1: Crystal_GND23, Crystals:Crystal_SMD_5032-4pin_5.0x3.2mm, F.Cu at (149.9, 124.0)
- C1: value C -> 4n7
- C12: value 0.1u -> 0.1
- C19: value 0.1 -> 4.7n
- C2, C3, C5, C9: value C -> 0.1
- C7: value 1u -> 1.0; footprint Capacitors_SMD:C_0603 -> Capacitors_SMD:C_0805
- C8: value 1u -> 0.1
- D3: value D -> D_Schottky
- J2: value Screw_Terminal_1x02 -> CONN_01X03; footprint Connectors_Terminal_Blocks:TerminalBlock_Pheonix_MKDS1.5-2pol -> Socket_Strips:Socket_Strip_Straight_1x03_Pitch2.54mm
- Q2, Q3: value Q_NMOS_GDS -> FQP30N06L
- R1, R4: value R -> 100R
- R10: value R -> 4.7K
- R12, R13: value R -> 0R1; footprint Resistors_THT:R_Axial_DIN0516_L15.5mm_D5.0mm_P20.32mm_Horizontal -> Resistors_SMD:R_2512
- R14: value R -> 10K; footprint Resistors_THT:R_Axial_DIN0516_L15.5mm_D5.0mm_P20.32mm_Horizontal -> Resistors_SMD:R_0603
- R15: value R -> 100K; footprint Resistors_THT:R_Axial_DIN0516_L15.5mm_D5.0mm_P20.32mm_Horizontal -> Resistors_SMD:R_0603
- R2: value R -> 24K
- R3, R9: value R -> 10K
- R5: value 90.9k -> 4.7K
- R6: value 8.45k -> 10K
- R7, R8: value R -> 100K
- RV1: value POT_TRIM -> POT; footprint Potentiometers:Potentiometer_Trimmer_Bourns_3214G -> Potentiometers:Potentiometer_Alps_RK09K_Horizontal
- SW1: footprint Buttons_Switches_THT:SW_SPDT -> Socket_Strips:Socket_Strip_Straight_1x02_Pitch2.54mm
- TP4: footprint Measurement_Points:Test_Point -> Measurement_Points:Measurement_Point_Round-TH_Big
- moved R16 126.1 mm to (184.8, 62.9), turned to 180 degrees
- moved C2 120.7 mm to (189.9, 62.9)
- moved C3 107.4 mm to (138.4, 67.9), turned to 270 degrees
- moved R11 103.2 mm to (136.5, 67.9), turned to 270 degrees
- moved C5 91.1 mm to (121.3, 85.1), turned to 90 degrees
- moved R4 89.3 mm to (120.7, 92.1), turned to 270 degrees
- moved RV1 89.0 mm to (118.1, 131.4), turned to 270 degrees
- moved R9 88.2 mm to (167.0, 90.2)
- moved J2 87.8 mm to (139.1, 105.4), turned to 315 degrees
- moved R8 80.6 mm to (163.8, 92.1)
- moved R3 79.3 mm to (162.6, 94.6), turned to 90 degrees
- moved C18 70.7 mm to (156.2, 86.4), turned to 180 degrees
- moved D2 69.2 mm to (130.2, 102.9), turned to 180 degrees
- moved TP4 67.1 mm to (165.1, 84.5)
- moved R10 63.5 mm to (167.0, 95.2)
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Connections:
- C1 pad 1: GND -> Net-(1M1-Pad1)
- C1 pad 2: (no net) -> GND
- C12 pad 1: +BATT -> /load_box_interface/STATIC_VREF
- C18 pad 1: +12V -> Net-(C18-Pad1)
- C19 pad 1: +12V -> /load_box_sink/REMOTE_SENSE_OUT
- C2 pad 1: GND -> Net-(C2-Pad1)
- C2 pad 2: +3V3 -> GND
- C3 pad 1: GND -> Net-(C3-Pad1)
- C3 pad 2: +3V3 -> GND
- C4 pad 1: (no net) -> Net-(C4-Pad1)
- C5 pad 1: +3V3 -> NRST
- C6 pad 1: (no net) -> Net-(C6-Pad1)
- C7 pad 1: +BATT -> Net-(C7-Pad1)
- C8 pad 1: /load_box_display/+13V -> Net-(C8-Pad1)
- C9 pad 1: USERB -> /load_box_interface/STEP_VREF
- C9 pad 2: Net-(C9-Pad2) -> GND
- D1 pad 1: Net-(D1-Pad1) -> +BATT
- D2 pad 1: GND -> +BATT
- D2 pad 2: Net-(D1-Pad1) -> +12V
- D3 pad 1: +12V -> +3V3
- D3 pad 2: Net-(D3-Pad2) -> /load_box_sink/REMOTE_SENSE_OUT
- J2 pad 1: Net-(J2-Pad1) -> GND
- Q2 pad 1: Net-(Q2-Pad1) -> Net-(C3-Pad1)
- Q3 pad 1: Net-(Q3-Pad1) -> Net-(C2-Pad1)
- R1 pad 1: +5V -> +3V3
- R1 pad 2: USERB -> Net-(C18-Pad1)
- R10 pad 1: Net-(Q1-Pad1) -> GND
- R11 pad 1: Net-(Q2-Pad1) -> Net-(C3-Pad1)
- R14 pad 1: Net-(Q2-Pad3) -> Net-(R10-Pad2)
- R14 pad 2: GND -> Net-(R14-Pad2)
- R15 pad 1: Net-(Q2-Pad3) -> Net-(R14-Pad2)
- R15 pad 2: GND -> /load_box_sink/REMOTE_SENSE_OUT
- R16 pad 1: Net-(Q3-Pad1) -> Net-(C2-Pad1)
- R2 pad 1: Net-(C9-Pad2) -> Net-(R2-Pad1)
- R2 pad 2: GND -> Net-(R2-Pad2)
- R3 pad 1: GND -> Net-(R2-Pad2)
- R3 pad 2: (no net) -> GND
- R4 pad 1: (no net) -> /load_box_interface/USER_BUTTON
- R4 pad 2: Net-(D1-Pad2) -> Net-(C8-Pad1)
- R5 pad 1: /load_box_display/+13V -> +3V3
- R5 pad 2: Net-(R5-Pad2) -> /load_box_interface/USER_BUTTON
- R6 pad 1: Net-(R5-Pad2) -> +3V3
- R6 pad 2: GND -> /load_box_interface/GO_BUTTON
- R7 pad 1: Net-(R20-Pad2) -> Net-(R7-Pad1)
- R7 pad 2: GND -> Net-(J5-Pad1)
- R8 pad 1: Net-(R8-Pad1) -> Net-(R10-Pad2)
- R8 pad 2: Net-(R8-Pad2) -> Net-(J5-Pad2)
- R9 pad 1: Net-(Q2-Pad3) -> Net-(R7-Pad1)
- R9 pad 2: Net-(R8-Pad1) -> GND
- RV1 pad 1: +12V -> +3V3
- RV1 pad 2: Net-(RV1-Pad2) -> /load_box_interface/STEP_VREF
- SW1 pad 2: +BATT -> +12V
- TP4 pad 1: +12V -> Net-(C18-Pad1)
- U1 pad 1: Net-(R8-Pad1) -> Net-(R2-Pad1)
- U1 pad 10: Net-(RV1-Pad2) -> Net-(R7-Pad1)
- U1 pad 11: GND -> (no net)
- U1 pad 12: (no net) -> /load_box_mcu/CHOSEN_VREF
- U1 pad 13: Net-(R8-Pad1) -> Net-(R2-Pad1)
- U1 pad 2: Net-(R8-Pad2) -> Net-(R2-Pad2)
- U1 pad 3: Net-(R20-Pad2) -> Net-(Q2-Pad3)
- U1 pad 4: +12V -> Net-(C18-Pad1)
- U1 pad 5: Net-(U1-Pad5) -> (no net)
- U1 pad 6: /load_box_mcu/MEASURED_VREF -> (no net)
- U1 pad 7: /load_box_mcu/MEASURED_VREF -> (no net)
- U1 pad 8: Net-(R10-Pad2) -> Net-(R14-Pad2)
- U1 pad 9: Net-(R18-Pad2) -> Net-(R10-Pad2)
- U4 pad 1: (no net) -> Net-(C7-Pad1)
- U4 pad 10: /load_box_mcu/MEASURED_VREF -> (no net)
- U4 pad 13: (no net) -> Net-(L2-Pad2)
- U4 pad 19: (no net) -> Net-(C14-Pad1)
- U4 pad 2: (no net) -> /load_box_interface/USER_BUTTON
- U4 pad 3: (no net) -> Net-(C4-Pad1)
- U4 pad 32: (no net) -> Net-(C15-Pad1)
- U4 pad 4: (no net) -> Net-(C6-Pad1)
- U4 pad 42: (no net) -> Net-(J2-Pad2)
- U4 pad 43: (no net) -> Net-(J2-Pad3)
- U4 pad 44: (no net) -> /load_box_mcu/USB_DM
- U4 pad 45: (no net) -> /load_box_mcu/USB_DP
- U4 pad 48: (no net) -> Net-(C16-Pad1)
- U4 pad 53: (no net) -> /load_box_display/MOSI
- U4 pad 64: (no net) -> Net-(C17-Pad1)
- U4 pad 7: (no net) -> NRST
- U4 pad 8: (no net) -> /load_box_interface/STATIC_VREF
- U4 pad 9: (no net) -> /load_box_interface/STEP_VREF
Routing:
- net GND: track 0.00 -> 171.1 mm, vias 0 -> 1
- net Net-(R11-Pad2): track 0.00 -> 102.3 mm, vias 0 -> 2
- net +3V3: track 0.00 -> 59.0 mm, vias 0 -> 5
- net /load_box_display/MOSI: track 0.00 -> 46.5 mm, vias 0 -> 1
- net Net-(Q2-Pad3): track 0.00 -> 43.3 mm, vias 0 -> 2
- net /load_box_interface/STEP_VREF: track 0.00 -> 36.2 mm, vias 0 -> 1
- net /load_box_interface/STATIC_VREF: track 0.00 -> 28.2 mm, vias 0 -> 3
- net +BATT: track 0.00 -> 26.9 mm
- net +12V: track 0.00 -> 25.3 mm, vias 0 -> 1
- net Net-(1M1-Pad1): track 0.00 -> 21.1 mm
- net Net-(C2-Pad1): track 0.00 -> 20.1 mm, vias 0 -> 1
- net Net-(C18-Pad1): track 0.00 -> 18.8 mm
- net /load_box_mcu/USB_DP: track 0.00 -> 18.2 mm
- net /load_box_mcu/USB_DM: track 0.00 -> 17.1 mm
- net Net-(J1-Pad1): track 0.00 -> 13.1 mm
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- added copper zone on F.Cu, net GND
- added copper zone on B.Cu, net Net-(J3-Pad1)
- added copper zone on F.Cu, net Net-(Q2-Pad3)
Other:
- board text added: "Fan"
- board text added: "Heatsink"
