File: class2.2/load_box_display.sch (KiCad schematic (older format))
At the start: 10 parts

Commit message: checkpoint some analog
Parts:
- C1, C2, C3, C5, C6: renamed from C?; footprint (none) -> Capacitors_SMD:C_0603
- D1, D2: renamed from D?; footprint (none) -> Diodes_SMD:D_SOD-123
- R3, R4: renamed from R?; footprint (none) -> Resistors_SMD:R_0603
- gave numbers to parts that had none: 1
Changed lines of the file:
@@
 LIBS:stm32
 LIBS:switches
-LIBS:fpc
 LIBS:load_box-cache
 EELAYER 25 0
@@
 $Descr A4 11693 8268
 encoding utf-8
-Sheet 2 7
+Sheet 2 6
 Title ""
 Date ""
@@
 $EndDescr
 $Comp
-L FPC-30 P?
+L FPC-30 P1
 U 1 1 58EFF997
 P 5200 3700
-F 0 "P?" H 5000 5600 60  0000 C CNN
+F 0 "P1" H 5000 5600 60  0000 C CNN
 F 1 "FPC-30" H 5100 2625 60  0000 C CNN
 F 2 "" H 5150 3700 60  0001 C CNN
@@
 $EndComp
 $Comp
-L GND #PWR?
+L GND #PWR10
 U 1 1 58EFFA17
 P 5950 2000
-F 0 "#PWR?" H 5950 1750 50  0001 C CNN
+F 0 "#PWR10" H 5950 1750 50  0001 C CNN
 F 1 "GND" H 5950 1850 50  0000 C CNN
 F 2 "" H 5950 2000 50  0001 C CNN
@@
 	6850 2100 5700 2100
 $Comp
-L GND #PWR?
+L GND #PWR11
 U 1 1 58EFFA94
 P 6650 3100
-F 0 "#PWR?" H 6650 2850 50  0001 C CNN
+F 0 "#PWR11" H 6650 2850 50  0001 C CNN
 F 1 "GND" H 6650 2950 50  0000 C CNN
 F 2 "" H 6650 3100 50  0001 C CNN
@@
 $EndComp
 $Comp
-L C C?
+L C C6
 U 1 1 58EFFAA3
 P 6800 2500
-F 0 "C?" H 6825 2600 50  0000 L CNN
+F 0 "C6" H 6825 2600 50  0000 L CNN
 F 1 "C" H 6825 2400 50  0000 L CNN
-F 2 "" H 6838 2350 50  0001 C CNN
+F 2 "Capacitors_SMD:C_0603" H 6838 2350 50  0001 C CNN
 F 3 "" H 6800 2500 50  0001 C CNN
 	1    6800 2500
@@
 $EndComp
 $Comp
-L C C?
+L C C5
 U 1 1 58EFFAC2
 P 6550 2500
-F 0 "C?" H 6575 2600 50  0000 L CNN
+F 0 "C5" H 6575 2600 50  0000 L CNN
 F 1 "C" H 6575 2400 50  0000 L CNN
-F 2 "" H 6588 2350 50  0001 C CNN
+F 2 "Capacitors_SMD:C_0603" H 6588 2350 50  0001 C CNN
 F 3 "" H 6550 2500 50  0001 C CNN
 	1    6550 2500
@@
 	6800 2200 6800 2350
 $Comp
-L +3.3V #PWR?
+L +3.3V #PWR14
 U 1 1 58EFFAF4
 P 6950 2300
-F 0 "#PWR?" H 6950 2150 50  0001 C CNN
+F 0 "#PWR14" H 6950 2150 50  0001 C CNN
 F 1 "+3.3V" H 6950 2440 50  0000 C CNN
 F 2 "" H 6950 2300 50  0001 C CNN
@@
 Connection ~ 6550 2300
 $Comp
-L D D?
+L D D1
 U 1 1 58EFFB58
 P 6300 2550
-F 0 "D?" H 6300 2650 50  0000 C CNN
+F 0 "D1" H 6300 2650 50  0000 C CNN
 F 1 "D" H 6300 2450 50  0000 C CNN
-F 2 "" H 6300 2550 50  0001 C CNN
+F 2 "Diodes_SMD:D_SOD-123" H 6300 2550 50  0001 C CNN
 F 3 "" H 6300 2550 50  0001 C CNN
 	1    6300 2550
@@
 $EndComp
 $Comp
-L D D?
+L D D2
 U 1 1 58EFFBF3
 P 6300 2900
-F 0 "D?" H 6300 3000 50  0000 C CNN
+F 0 "D2" H 6300 3000 50  0000 C CNN
 F 1 "D" H 6300 2800 50  0000 C CNN
-F 2 "" H 6300 2900 50  0001 C CNN
+F 2 "Diodes_SMD:D_SOD-123" H 6300 2900 50  0001 C CNN
 F 3 "" H 6300 2900 50  0001 C CNN
 	1    6300 2900
@@
 	6300 2750 6300 2700
 $Comp
-L R R?
+L R R4
 U 1 1 58EFFC7A
 P 6000 2400
-F 0 "R?" V 6080 2400 50  0000 C CNN
+F 0 "R4" V 6080 2400 50  0000 C CNN
 F 1 "R" V 6000 2400 50  0000 C CNN
-F 2 "" V 5930 2400 50  0001 C CNN
+F 2 "Resistors_SMD:R_0603" V 5930 2400 50  0001 C CNN
 F 3 "" H 6000 2400 50  0001 C CNN
 	1    6000 2400
@@
 	6000 4000 5700 4000
 $Comp
-L R R?
+L R R3
 U 1 1 58F0008A
 P 5950 4100
-F 0 "R?" V 6030 4100 50  0000 C CNN
+F 0 "R3" V 6030 4100 50  0000 C CNN
 F 1 "R" V 5950 4100 50  0000 C CNN
-F 2 "" V 5880 4100 50  0001 C CNN
+F 2 "Resistors_SMD:R_0603" V 5880 4100 50  0001 C CNN
 F 3 "" H 5950 4100 50  0001 C CNN
 	1    5950 4100
@@
 	5800 4100 5700 4100
 $Comp
-L C C?
+L C C2
 U 1 1 58F0013F
 P 6200 4450
-F 0 "C?" H 6225 4550 50  0000 L CNN
+F 0 "C2" H 6225 4550 50  0000 L CNN
 F 1 "C" H 6225 4350 50  0000 L CNN
-F 2 "" H 6238 4300 50  0001 C CNN
+F 2 "Capacitors_SMD:C_0603" H 6238 4300 50  0001 C CNN
 F 3 "" H 6200 4450 50  0001 C CNN
 	1    6200 4450
@@
 $EndComp
 $Comp
-L C C?
+L C C3
 U 1 1 58F001DC
 P 6450 4450
-F 0 "C?" H 6475 4550 50  0000 L CNN
+F 0 "C3" H 6475 4550 50  0000 L CNN
 F 1 "C" H 6475 4350 50  0000 L CNN
-F 2 "" H 6488 4300 50  0001 C CNN
+F 2 "Capacitors_SMD:C_0603" H 6488 4300 50  0001 C CNN
 F 3 "" H 6450 4450 50  0001 C CNN
 	1    6450 4450
@@
 Connection ~ 6200 4600
 $Comp
-L +3.3V #PWR?
+L +3.3V #PWR13
 U 1 1 58F0024F
 P 6700 4600
-F 0 "#PWR?" H 6700 4450 50  0001 C CNN
+F 0 "#PWR13" H 6700 4450 50  0001 C CNN
 F 1 "+3.3V" H 6700 4740 50  0000 C CNN
 F 2 "" H 6700 4600 50  0001 C CNN
@@
 	6450 4300 6450 4100
 $Comp
-L GND #PWR?
+L GND #PWR12
 U 1 1 58F0033A
 P 6700 4300
-F 0 "#PWR?" H 6700 4050 50  0001 C CNN
+F 0 "#PWR12" H 6700 4050 50  0001 C CNN
 F 1 "GND" H 6700 4150 50  0000 C CNN
 F 2 "" H 6700 4300 50  0001 C CNN
@@
 $EndComp
 $Comp
-L GND #PWR?
+L GND #PWR9
 U 1 1 58F003A8
 P 5850 5050
-F 0 "#PWR?" H 5850 4800 50  0001 C CNN
+F 0 "#PWR9" H 5850 4800 50  0001 C CNN
 F 1 "GND" H 5850 4900 50  0000 C CNN
 F 2 "" H 5850 5050 50  0001 C CNN
@@
 	6000 3600 5700 3600
 $Comp
-L GND #PWR?
+L GND #PWR8
 U 1 1 58F00650
 P 5850 3500
-F 0 "#PWR?" H 5850 3250 50  0001 C CNN
+F 0 "#PWR8" H 5850 3250 50  0001 C CNN
 F 1 "GND" H 5850 3350 50  0000 C CNN
 F 2 "" H 5850 3500 50  0001 C CNN
@@
 Connection ~ 5850 3500
 $Comp
-L GND #PWR?
+L GND #PWR7
 U 1 1 58F00678
 P 5800 3900
-F 0 "#PWR?" H 5800 3650 50  0001 C CNN
+F 0 "#PWR7" H 5800 3650 50  0001 C CNN
 F 1 "GND" H 5800 3750 50  0000 C CNN
 F 2 "" H 5800 3900 50  0001 C CNN
@@
 Series cap looks wrong, but pin 26 is regulated from VCI on pin 27
 $Comp
-L C C?
+L C C1
 U 1 1 58F009DF
 P 6000 4300
-F 0 "C?" H 6025 4400 50  0000 L CNN
+F 0 "C1" H 6025 4400 50  0000 L CNN
 F 1 "C" H 6025 4200 50  0000 L CNN
-F 2 "" H 6038 4150 50  0001 C CNN
+F 2 "Capacitors_SMD:C_0603" H 6038 4150 50  0001 C CNN
 F 3 "" H 6000 4300 50  0001 C CNN
 	1    6000 4300

Commit message: Checkpoint with NHD, 3.3v, and layout
Parts:
- removed C1, C2, C3, C5, C6: C, Capacitors_SMD:C_0603, symbol C
- removed D1, D2: D, Diodes_SMD:D_SOD-123, symbol D
- removed P1: FPC-30, symbol FPC-30
- removed R3, R4: R, Resistors_SMD:R_0603, symbol R
- added J4: CONN_02X10, nhd:NHD-1.69, symbol CONN_02X10
Connections:
- net +3V3: now also J4.2 (P2)
- net GND: now also J4.1 (P1), J4.10 (P10), J4.11 (P11), J4.12 (P12), J4.15 (P15), J4.18 (P18), J4.19 (P19), J4.20 (P20), J4.5 (P5), J4.6 (P6), J4.7 (P7), J4.8 (P8), J4.9 (P9)
- net MOSI: now also J4.13 (P13)
- net SCLK: now also J4.14 (P14)
- net ~CS: now also J4.17 (P17)
- new net RS: J4.4 (P4)
- new net ~RES: J4.16 (P16)
- no-connect marks 6 -> 1
Other:
- note removed: "NOTE:\nObserve proper direction of FPC cable, footprint supports both top and bottom contact parts."
- note removed: "Series cap looks wrong, but pin 26 is regulated from VCI on pin 27"
