File: class2.2/load_box_interface.sch (KiCad schematic (older format))
At the start: 0 parts

Commit message: Checkpoint with NHD, 3.3v, and layout
Parts:
- added C12, C8, C9: 0.1, Capacitors_SMD:C_0603, symbol C
- added C13: 0.1, symbol C
- added R6: 10K, Resistors_SMD:R_0603, symbol R
- added RV1, RV2: POT, Potentiometers:Potentiometer_Alps_RK09K_Horizontal, symbol POT
- added SW3: SW_Push, Buttons_Switches_THT:SW_Tactile_SKHH_Angled, symbol SW_Push
- added SW4: SW_Push, Pin_Headers:Pin_Header_Straight_1x02_Pitch2.54mm, symbol SW_Push
Connections:
- new net +3V3: C8.1, R6.1, RV1.1, RV2.1, SW3.1
- new net BOOT0: C8.2, SW3.2
- new net GND: C12.2, C13.2, C9.2, RV1.3, RV2.3, SW4.1
- new net GO_BUTTON: C13.1, R6.2, SW4.2
- new net STATIC_VREF: C12.1, RV2.2
- new net STEP_VREF: C9.1, RV1.2
Other:
- note added: "BOOT0 controls whether\nUSB bootloader runs on\npowerup."
- note added: "Note: These go into ADC, and are not used directly."
- note added: "See STM32 Nucleo schematics\nfor recommended minimum\nsystem board."
- note added: "http://www.st.com/en/evaluation-tools/nucleo-l152re.html"
