File: class2.2/load_box_mcu.sch (KiCad schematic (older format))
At the start: 0 parts

Commit message: Snapshot with basic MCU, analog
Parts:
- added C? (x4): C, symbol C
- added J?: USB_B, symbol USB_B
- added L?: Ferrite_Bead, symbol Ferrite_Bead
- added TP? (x4): TEST, symbol TEST
- added U?: STM32L152RCTx, LQFP64, symbol STM32L152RCTx
Connections:
- new net: L?.2, U?.13 (VDDA)
- new net: C?.1, U?.19 (VDD)
- new net: C?.1, U?.32 (VDD)
- new net: TP?.1, U?.42 (DAC_EXTI9/LCD_COM1/TIMX_IC2/TS_G4_IO2/USART1_TX/PA9)
- new net: TP?.1, U?.43 (LCD_COM2/TIMX_IC3/TS_G4_IO3/USART1_RX/PA10)
- new net: J?.2 (D-), U?.44 (ADC_EXTI11/SPI1_MISO/TIMX_IC4/USART1_CTS/USB_DM/PA11)
- new net: J?.3 (D+), U?.45 (SPI1_MOSI/TIMX_IC1/USART1_RTS/USB_DP/PA12)
- new net: C?.1, U?.48 (VDD)
- new net: C?.1, U?.64 (VDD)
- new net +3V3: C?.2, C?.2, C?.2, C?.2, L?.1, TP?.1
- new net CHOSEN_VREF: U?.40 (PC9/DAC_EXTI9/LCD_SEG27/TIM3_CH4/TIMX_IC2/TS_G10_IO4)
- new net GND: J?.4 (GND), J?.5 (Shield), TP?.1, U?.12 (VSSA), U?.18 (VSS), U?.31 (VSS), U?.47 (VSS), U?.63 (VSS)
- new net MEASURED_VREF: U?.10 (PC2/ADC_IN12/COMP1_INP/LCD_SEG20/TIMX_IC3/TS_G8_IO3)
- new net OLED_CS: U?.39 (PC8/LCD_SEG26/TIM3_CH3/TIMX_IC1/TS_G10_IO3)
- new net OLED_MOSI: U?.53 (PC12/I2S3_SD/LCD_COM6/LCD_SEG30/LCD_SEG42/SPI3_MOSI/TIMX_IC1/USART3_CK)
- new net OLED_SCK: U?.51 (PC10/I2S3_CK/LCD_COM4/LCD_SEG28/LCD_SEG40/SPI3_SCK/TIMX_IC3/USART3_TX)
- new net STATIC_VREF: U?.8 (PC0/ADC_IN10/COMP1_INP/LCD_SEG18/TIMX_IC1/TS_G8_IO1)
- new net STEP_VREF: U?.9 (PC1/ADC_IN11/COMP1_INP/LCD_SEG19/TIMX_IC2/TS_G8_IO2)
- new net TEMPERATURE: U?.11 (PC3/ADC_IN13/COMP1_INP/LCD_SEG21/TIMX_IC4/TS_G8_IO4)
- new net ~OLED_RESET: U?.38 (PC7/I2S3_MCK/LCD_SEG25/TIM3_CH2/TIMX_IC4/TS_G10_IO2)
- no-connect marks 0 -> 1
Other:
- note added: "TODO 1m and cap shield per... atmel? or ftdi?"
- note added: "TODO 3.3v reg off this w/o wall power?"
- note added: "TODO DM/DP mapping?"
- note added: "TODO SWD header and pogo (is there a standard for either?)"
- note added: "TODO VSSA get a ferrite or anything?"
- note added: "TODO over power light?"
- note added: "TODO reset/user button"
- note added: "TODO total voltage, incl remote sense"
- note added: "TODO watch xtal?"
- note added: "TODO: ferrite?"

Commit message: Further layout.
Parts:
- U4: renamed from U?; footprint LQFP64 -> Housings_QFP:LQFP-64_10x10mm_Pitch0.5mm
- gave numbers to parts that had none: 10
Changed lines of the file:
@@
 LIBS:stm32
 LIBS:switches
+LIBS:fpc
+LIBS:ap3012
 LIBS:load_box-cache
 EELAYER 25 0
@@
 $EndDescr
 $Comp
-L STM32L152RCTx U?
+L STM32L152RCTx U4
 U 1 1 58F3E6A5
 P 5700 3200
-F 0 "U?" H 1900 5125 50  0000 L BNN
+F 0 "U4" H 1900 5125 50  0000 L BNN
 F 1 "STM32L152RCTx" H 9500 5125 50  0000 R BNN
-F 2 "LQFP64" H 9500 5075 50  0001 R TNN
+F 2 "Housings_QFP:LQFP-64_10x10mm_Pitch0.5mm" H 9500 5075 50  0001 R TNN
 F 3 "" H 5700 3200 50  0001 C CNN
 	1    5700 3200
@@
 $EndComp
 $Comp
-L Ferrite_Bead L?
+L Ferrite_Bead L2
 U 1 1 58F3E75A
 P 5900 1050
-F 0 "L?" V 5750 1075 50  0000 C CNN
+F 0 "L2" V 5750 1075 50  0000 C CNN
 F 1 "Ferrite_Bead" V 6050 1050 50  0000 C CNN
 F 2 "" V 5830 1050 50  0001 C CNN
@@
 $EndComp
 $Comp
-L C C?
+L C C14
 U 1 1 58F3E78D
 P 5500 1050
-F 0 "C?" H 5525 1150 50  0000 L CNN
+F 0 "C14" H 5525 1150 50  0000 L CNN
 F 1 "C" H 5525 950 50  0000 L CNN
 F 2 "" H 5538 900 50  0001 C CNN
@@
 $EndComp
 $Comp
-L C C?
+L C C15
 U 1 1 58F3E827
 P 5600 1050
-F 0 "C?" H 5625 1150 50  0000 L CNN
+F 0 "C15" H 5625 1150 50  0000 L CNN
 F 1 "C" H 5625 950 50  0000 L CNN
 F 2 "" H 5638 900 50  0001 C CNN
@@
 $EndComp
 $Comp
-L C C?
+L C C16
 U 1 1 58F3E847
 P 5700 1050
-F 0 "C?" H 5725 1150 50  0000 L CNN
+F 0 "C16" H 5725 1150 50  0000 L CNN
 F 1 "C" H 5725 950 50  0000 L CNN
 F 2 "" H 5738 900 50  0001 C CNN
@@
 $EndComp
 $Comp
-L C C?
+L C C17
 U 1 1 58F3E86A
 P 5800 1050
-F 0 "C?" H 5825 1150 50  0000 L CNN
+F 0 "C17" H 5825 1150 50  0000 L CNN
 F 1 "C" H 5825 950 50  0000 L CNN
 F 2 "" H 5838 900 50  0001 C CNN
@@
 $EndComp
 $Comp
-L +3.3V #PWR?
+L +3.3V #PWR048
 U 1 1 58F3E8AC
 P 5700 750
-F 0 "#PWR?" H 5700 600 50  0001 C CNN
+F 0 "#PWR048" H 5700 600 50  0001 C CNN
 F 1 "+3.3V" H 5700 890 50  0000 C CNN
 F 2 "" H 5700 750 50  0001 C CNN
@@
 	5500 900  5500 750
 Wire Wire Line
-	5500 750  5600 750
-Wire Wire Line
-	5600 750  5700 750
-Wire Wire Line
-	5700 750  5800 750
-Wire Wire Line
-	5800 750  5900 750
+	5500 750  5900 750
 Wire Wire Line
 	5900 750  5900 900
@@
 	9600 2800 10750 2800
 $Comp
-L USB_B J?
+L USB_B J5
 U 1 1 58F3FFA1
 P 10300 1900
-F 0 "J?" H 10100 2350 50  0000 L CNN
+F 0 "J5" H 10100 2350 50  0000 L CNN
 F 1 "USB_B" H 10100 2250 50  0000 L CNN
 F 2 "" H 10450 1850 50  0001 C CNN
@@
 TODO 3.3v reg off this w/o wall power?
 $Comp
-L GND #PWR?
+L GND #PWR049
 U 1 1 58F40095
 P 10200 2450
-F 0 "#PWR?" H 10200 2200 50  0001 C CNN
+F 0 "#PWR049" H 10200 2200 50  0001 C CNN
 F 1 "GND" H 10200 2300 50  0000 C CNN
 F 2 "" H 10200 2450 50  0001 C CNN
@@
 $EndComp
 Wire Wire Line
-	10200 2300 10200 2350
-Wire Wire Line
-	10200 2350 10200 2450
+	10200 2300 10200 2450
 Wire Wire Line
 	10200 2350 10300 2350
@@
 TODO SWD header and pogo (is there a standard for either?)
 $Comp
-L GND #PWR?
+L GND #PWR050
 U 1 1 58F404EF
 P 5700 5450
-F 0 "#PWR?" H 5700 5200 50  0001 C CNN
+F 0 "#PWR050" H 5700 5200 50  0001 C CNN
 F 1 "GND" H 5700 5300 50  0000 C CNN
 F 2 "" H 5700 5450 50  0001 C CNN
@@
 	5500 5200 5500 5350
 Wire Wire Line
-	5500 5350 5600 5350
-Wire Wire Line
-	5600 5350 5700 5350
-Wire Wire Line
-	5700 5350 5800 5350
-Wire Wire Line
-	5800 5350 5900 5350
+	5500 5350 5900 5350
 Wire Wire Line
 	5800 5350 5800 5200
 Wire Wire Line
-	5700 5200 5700 5350
-Wire Wire Line
-	5700 5350 5700 5450
+	5700 5200 5700 5450
 Wire Wire Line
 	5600 5200 5600 5350
@@
 TODO total voltage, incl remote sense
 $Comp
-L TEST TP?
+L TEST TP9
 U 1 1 58F41CC1
 P 9700 2500
-F 0 "TP?" H 9700 2800 50  0000 C BNN
+F 0 "TP9" H 9700 2800 50  0000 C BNN
 F 1 "TEST" H 9700 2750 50  0000 C CNN
 F 2 "" H 9700 2500 50  0001 C CNN
@@
 $EndComp
 $Comp
-L TEST TP?
+L TEST TP10
 U 1 1 58F41CFC
 P 9700 2600
-F 0 "TP?" H 9700 2900 50  0000 C BNN
+F 0 "TP10" H 9700 2900 50  0000 C BNN
 F 1 "TEST" H 9700 2850 50  0000 C CNN
 F 2 "" H 9700 2600 50  0001 C CNN
@@
 	9600 2600 9700 2600
 $Comp
-L GND #PWR?
+L GND #PWR051
 U 1 1 58F41EAD
 P 9950 2150
-F 0 "#PWR?" H 9950 1900 50  0001 C CNN
+F 0 "#PWR051" H 9950 1900 50  0001 C CNN
 F 1 "GND" H 9950 2000 50  0000 C CNN
 F 2 "" H 9950 2150 50  0001 C CNN
@@
 $EndComp
 $Comp
-L TEST TP?
+L TEST TP12
 U 1 1 58F41ED3
 P 9950 2150
-F 0 "TP?" H 9950 2450 50  0000 C BNN
+F 0 "TP12" H 9950 2450 50  0000 C BNN
 F 1 "TEST" H 9950 2400 50  0000 C CNN
 F 2 "" H 9950 2150 50  0001 C CNN
@@
 $EndComp
 $Comp
-L +3.3V #PWR?
+L +3.3V #PWR052
 U 1 1 58F4209F
 P 9800 2050
-F 0 "#PWR?" H 9800 1900 50  0001 C CNN
+F 0 "#PWR052" H 9800 1900 50  0001 C CNN
 F 1 "+3.3V" H 9800 2190 50  0000 C CNN
 F 2 "" H 9800 2050 50  0001 C CNN
@@
 $EndComp
 $Comp
-L TEST TP?
+L TEST TP11
 U 1 1 58F42136
 P 9800 2050
-F 0 "TP?" H 9800 2350 50  0000 C BNN
+F 0 "TP11" H 9800 2350 50  0000 C BNN
 F 1 "TEST" H 9800 2300 50  0000 C CNN
 F 2 "" H 9800 2050 50  0001 C CNN

Commit message: Checkpoint with NHD, 3.3v, and layout
Parts:
- removed J5: USB_B, symbol USB_B
- removed TP10, TP11, TP12, TP9: TEST, symbol TEST
- added C4, C6: C, Capacitors_SMD:C_0603, symbol C
- added C5: 0.1, Capacitors_SMD:C_0603, symbol C
- added C7: 1.0, Capacitors_SMD:C_0805, symbol C
- added J2: CONN_01X03, Socket_Strips:Socket_Strip_Straight_1x03_Pitch2.54mm, symbol CONN_01X03
- added SW2: SW_Push, Buttons_Switches_THT:SW_Tactile_SKHH_Angled, symbol SW_Push
- added Y1: Crystal_GND23, Crystals:Crystal_SMD_5032-4pin_5.0x3.2mm, symbol Crystal_GND23
- C14, C15, C16, C17: footprint (none) -> Capacitors_SMD:C_0603
- L2: footprint (none) -> Inductors_SMD:L_0603
Connections:
- net GND: now also C4.2, C5.2, C6.2, C7.2, J2.1 (P1), SW2.1
- net at U4.1 (VLCD): now also C7.1
- net at U4.3 (PC14/RCC_OSC32_IN/TIMX_IC3): now also C4.1, Y1.1
- net at U4.4 (PC15/ADC_EXTI15/RCC_OSC32_OUT/TIMX_IC4): now also C6.1, Y1.4
- net at U4.42 (DAC_EXTI9/LCD_COM1/TIMX_IC2/TS_G4_IO2/USART1_TX/PA9): now also J2.2 (P2)
- net at U4.43 (LCD_COM2/TIMX_IC3/TS_G4_IO3/USART1_RX/PA10): now also J2.3 (P3)
- net USB_DM: now reaches U4.44 (ADC_EXTI11/SPI1_MISO/TIMX_IC4/USART1_CTS/USB_DM/PA11)
- net USB_DP: now reaches U4.45 (SPI1_MOSI/TIMX_IC1/USART1_RTS/USB_DP/PA12)
- net TMS: now reaches U4.46 (SYS_JTMS-SWDIO/TIMX_IC2/TS_G5_IO1/PA13)
- net TCK: now reaches U4.49 (SYS_JTCK-SWCLK/TIMX_IC3/TS_G5_IO2/PA14)
- net SWO: now reaches U4.55 (COMP2_INM/I2S3_CK/LCD_SEG7/SPI1_SCK/SPI3_SCK/SYS_JTDO-TRACESWO/TIM2_CH2/PB3)
- net BOOT0: now reaches U4.60 (BOOT0)
- net NRST: now reaches U4.7 (NRST)
- net NRST: now also C5.1, SW2.2
- no-connect marks 1 -> 0
Other:
- note added: "Serial header"
- note added: "TODO blinky LED on\nwhatever pin nucleo uses"
- note added: "TODO make sure ADC channels\nare not multipliexed"
- note removed: "TODO 1m and cap shield per... atmel? or ftdi?"
- note removed: "TODO 3.3v reg off this w/o wall power?"
- note removed: "TODO DM/DP mapping?"
- note removed: "TODO SWD header and pogo (is there a standard for either?)"
- note removed: "TODO VSSA get a ferrite or anything?"
- note removed: "TODO over power light?"
- note removed: "TODO reset/user button"
