File: class2.2/load_box_power.sch (KiCad schematic (older format))
At the start: 0 parts

Commit message: Moving class2.2 forward, includes 13V switching converter.
Parts:
- added C10: 0.1u, Capacitors_SMD:C_0603, symbol C
- added C11: 10u, Capacitors_SMD:C_1206, symbol C
- added C7, C8: 1u, symbol C
- added D3: 1N5819, symbol D_Schottky
- added J1: BARREL_JACK, Connectors:JACK_ALIM, symbol BARREL_JACK
- added L1: 10uH, Inductors_SMD:L_Wuerth_MAPI-2510, symbol L
- added R5: 90.9k, Resistors_SMD:R_0603, symbol R
- added R6: 8.45k, Resistors_SMD:R_0603, symbol R
- added SW1: SW_SPST, Buttons_Switches_THT:SW_SPDT, symbol SW_SPST
- added U1: AP3012, TO_SOT_Packages_SMD:SOT-23-5, symbol AP3012
- added U2: LD1117S33TR, TO_SOT_Packages_SMD:SOT-223, symbol LD1117S33TR
Connections:
- new net: J1.1, SW1.1 (A)
- new net: D3.2 (A), L1.2, U1.1 (SW)
- new net: R5.2, R6.1, U1.3 (FB)
- new net +12V: C10.1, C7.1, L1.1, SW1.2 (B), U1.5 (V_in), U2.3 (VI)
- new net +13V: C8.1, D3.1 (K), R5.1
- new net +3V3: C11.1, U1.4 (~SHDN), U2.2 (VO)
- new net GND: C10.2, C11.2, C7.2, C8.2, J1.2, J1.3, R6.2, U1.2 (GND), U2.1 (GND)
Other:
- note added: "12V nominal, center positive"
- note added: "Microcontroller is 3.3V"

Commit message: Further layout.
Parts:
- added C12: 0.1u, Capacitors_SMD:C_0603, symbol C
- added C13: 10u, Capacitors_SMD:C_1206, symbol C
- added J4: CONN_01X05, symbol CONN_01X05
- added R17: 10K, symbol R
- added U3: LD1117S50TR, TO_SOT_Packages_SMD:SOT-223, symbol LD1117S50TR
- J1: footprint Connectors:JACK_ALIM -> Connectors:BARREL_JACK
- renumbered D3 to D4, U1 to U5, U2 to U6
Connections:
- net +13V: now also J4.3 (P3)
- net +3V3: now also J4.5 (P5); no longer U5.4 (~SHDN)
- net GND: now also C12.2, C13.2, J4.1 (P1), U3.1 (GND)
- net +12V renamed +BATT
- net +BATT: now also C12.1, R17.1, U3.3 (VI)
- new net: R17.2, U5.4 (~SHDN)
- new net +5V: C13.1, J4.4 (P4), U3.2 (VO)
Other:
- note added: "Extra supply for op-amps and mosfet drive\n(consider removing in next rev if not required)"
- note added: "Note: AP3012 and LMR62014X are pin-compatible,\nbut AP3012 input voltage can be much higher."
- note added: "TODO: Tap on, long press off circuit?"
- note added: "TODO: Verify Vin > Vout does something sensible."
- note added: "TODO: Verify that this can start up after +3.3V\nand display will be ok."
- note added: "Test pins"
- moved on the sheet: C10, C11, C7, C8, D4, L1, R5, R6, U5, U6

Commit message: Checkpoint with NHD, 3.3v, and layout
Parts:
- removed C12: 0.1u, Capacitors_SMD:C_0603, symbol C
- removed C13: 10u, Capacitors_SMD:C_1206, symbol C
- removed C7, C8: 1u, symbol C
- removed D4: 1N5819, symbol D_Schottky
- removed J4: CONN_01X05, symbol CONN_01X05
- removed L1: 10uH, Inductors_SMD:L_Wuerth_MAPI-2510, symbol L
- removed R17: 10K, symbol R
- removed R5: 90.9k, Resistors_SMD:R_0603, symbol R
- removed R6: 8.45k, Resistors_SMD:R_0603, symbol R
- removed U3: LD1117S50TR, TO_SOT_Packages_SMD:SOT-223, symbol LD1117S50TR
- removed U5: AP3012, TO_SOT_Packages_SMD:SOT-23-5, symbol AP3012
- added 1M1: R, Resistors_SMD:R_0603, symbol R
- added C1: 4n7, Capacitors_SMD:C_0603, symbol C
- added D1, D2: D, Diodes_SMD:D_SOD-123, symbol D
- added J7: USB_B, Connectors:USB_B, symbol USB_B
- added J8: CONN_01X03, Socket_Strips:Socket_Strip_Straight_1x03_Pitch2.54mm, symbol CONN_01X03
- SW1: footprint Buttons_Switches_THT:SW_SPDT -> Socket_Strips:Socket_Strip_Straight_1x02_Pitch2.54mm
Connections:
- net +3V3: now also J8.3 (P3)
- net +BATT: now also D1.1 (K), D2.1 (K), J8.2 (P2); no longer SW1.2 (B)
- net GND: now also 1M1.2, C1.2, J7.4 (GND), J8.1 (P1)
- new net: D1.2 (A), J7.1 (VBUS)
- new net: 1M1.1, C1.1, J7.5 (Shield)
- new net +12V: D2.2 (A), SW1.2 (B)
- new net USB_DM: J7.2 (D-)
- new net USB_DP: J7.3 (D+)
Other:
- note added: "(Only used for fan)"
- note added: "Notes:\n- OLED draw is about 140mA\n- MCU draw is ???\n- Op-Amp draw is ???\n"
- note added: "Reverse-blocking diodes\nallow programming if you\nforget to switch power off.\n\nDiode drop is acceptable\nfrom 4.5V supply, we only\nneed about 3.8V for LDO"
- note removed: "Extra supply for op-amps and mosfet drive\n(consider removing in next rev if not required)"
- note removed: "Note: AP3012 and LMR62014X are pin-compatible,\nbut AP3012 input voltage can be much higher."
- note removed: "TODO: Tap on, long press off circuit?"
- note removed: "TODO: Verify Vin > Vout does something sensible."
- note removed: "TODO: Verify that this can start up after +3.3V\nand display will be ok."
- moved on the sheet: C10, C11, J1, U6
