File: class2.2/load_box_sink.sch (KiCad schematic (older format))
At the start: 0 parts

Commit message: checkpoint some analog
Parts:
- added C7, C8: 0.1, Capacitors_SMD:C_0603, symbol C
- added D3: D, Diodes_SMD:D_SOD-123, symbol D
- added J1: CONN_01X02, Connectors_JST:JST_XH_B02B-XH-A_02x2.50mm_Straight, symbol CONN_01X02
- added J2, J3: Screw_Terminal_1x02, Connectors_Terminal_Blocks:TerminalBlock_Pheonix_MKDS1.5-2pol, symbol Screw_Terminal_1x02
- added Q1: Q_NMOS_GDS, TO_SOT_Packages_SMD:SOT-23, symbol Q_NMOS_GDS
- added Q2, Q3: Q_NMOS_GDS, TO_SOT_Packages_THT:TO-220_Vertical, symbol Q_NMOS_GDS
- added R10, R19, R23, R24, R25, R26, R5, R6, R7, R8, R9: R, Resistors_SMD:R_0603, symbol R
- added R11, R16: 100R, Resistors_SMD:R_0603, symbol R
- added R12, R13, R14, R15: R, Resistors_THT:R_Axial_DIN0516_L15.5mm_D5.0mm_P20.32mm_Horizontal, symbol R
- added RV1: POT_TRIM, Potentiometers:Potentiometer_Trimmer_Bourns_3214G, symbol POT_TRIM
- added TH1: Thermistor_NTC, Connectors_JST:JST_XH_B02B-XH-A_02x2.50mm_Straight, symbol Thermistor_NTC
- added TP1, TP2, TP3, TP4, TP5, TP6, TP7, TP8: TEST, Measurement_Points:Test_Point, symbol TEST
- added U1: LM324, Housings_SOIC:SOIC-14_3.9x8.7mm_Pitch1.27mm, symbol LM324
- added U2: INA128, Housings_SOIC:SOIC-8_3.9x4.9mm_Pitch1.27mm, symbol INA128
Connections:
- new net: Q2.3 (S), Q3.3 (S), R12.1, R13.1, R14.1, R15.1, R9.1
- new net: J2.1, R23.1
- new net: J2.2, R25.2, R26.1
- new net: R23.2, R24.1, TP6.1, U2.3 (+)
- new net: R24.2, R25.1, TP7.1, U2.2 (-)
- new net: R8.1, R9.2, TP3.1, U1.1, U1.13 (-)
- new net: R11.2, R16.2, U1.14
- new net: R8.2, U1.2 (-)
- new net: R6.2, R7.1, TP2.1, U1.3 (+)
- new net: U1.5 (+), U2.6
- new net: RV1.2, U1.10 (+)
- new net: R10.2, U1.8
- new net: R5.2, TH1.1, U1.9 (-)
- new net: J3.1, Q2.2 (D), Q3.2 (D)
- new net: Q2.1 (G), R11.1, TP5.1
- new net: R19.1, U2.1 (Rg)
- new net: R19.2, U2.8 (Rg)
- new net: D3.2 (A), J1.2 (P2), Q1.2 (D)
- new net: Q1.1 (G), R10.1
- new net: Q3.1 (G), R16.1, TP8.1
- new net +12V: C7.1, C8.1, D3.1 (K), J1.1 (P1), R5.1, RV1.1, TP4.1, U1.4 (V+), U2.7 (V+)
- new net CHOSEN_VREF: R6.1, TP1.1
- new net GND: C7.2, C8.2, J3.2, Q1.3 (S), R12.2, R13.2, R14.2, R15.2, R26.2, R7.2, RV1.3, TH1.2, U1.11 (V-), U2.4 (V-), U2.5 (Ref)
- new net MEASURED_VREF: U1.6 (-), U1.7
Other:
- note added: "Buffer out of an\nabundance of caution\n(INA is expensive)"
- note added: "Main Load"
- note added: "Remote sense"
- note added: "TODO: 5V supply for analog"
- note added: "TODO: Ensure this is 3.3V max (and that we get 30-100C full range)"
- note added: "TODO: Ensures there is a common ground?\nDoes INA behave without it, or with\na super weak pulldown after the symmetric divider"
- note added: "TODO: Low current grounds tie together\nTODO: Place AGND a diode drop lower than this screw term?"
- note added: "TODO: Maybe just series resistor?"
- note added: "TODO: add resistors to make trim pot\nmore useful"
- note added: "TODO: damp output a lot"
- note added: "TODO: look up standard circuit where input may be 36V"
- note added: "TODO: resistor values for 3.3V = 6.6A,\nhere and shunt."
- note added: "TODO: simulate and reduce oscillations"
- note added: "TODO: verify whether paralleled resistor useful for log scale, NYC side"
- note added: "TODO: zener to restrict +\nTODO: reverse protection"

Commit message: Snapshot with basic MCU, analog
Other:
- note added: "TODO Rename this for the fact\nit's just scaked voltage across\nthe terminals, and not anything\nto do with current."
- note added: "TODO diodes vs the main connector as in a PSU?"
Changed lines of the file:
@@
 	5800 2850 5800 3050
 Connection ~ 5800 3050
+Text Notes 2400 4850 0    60   ~ 0
+TODO Rename this for the fact\nit's just scaked voltage across\nthe terminals, and not anything\nto do with current.
+Text Notes 7450 4900 0    60   ~ 0
+TODO diodes vs the main connector as in a PSU?
 $EndSCHEMATC

Commit message: Further layout.
Parts:
- renumbered C7 to C18, C8 to C19, J1 to J6, R5 to R18, R6 to R20
Changed lines of the file:
@@
 LIBS:stm32
 LIBS:switches
+LIBS:fpc
+LIBS:ap3012
 LIBS:load_box-cache
 EELAYER 25 0
@@
 	3250 3250 3650 3250
 $Comp
-L R R6
+L R R20
 U 1 1 58F1EF26
 P 3250 3000
-F 0 "R6" V 3330 3000 50  0000 C CNN
+F 0 "R20" V 3330 3000 50  0000 C CNN
 F 1 "R" V 3250 3000 50  0000 C CNN
 F 2 "Resistors_SMD:R_0603" V 3180 3000 50  0001 C CNN
@@
 	3250 2750 3250 2850
 $Comp
-L GND #PWR17
+L GND #PWR015
 U 1 1 58F1F160
 P 3250 3750
-F 0 "#PWR17" H 3250 3500 50  0001 C CNN
+F 0 "#PWR015" H 3250 3500 50  0001 C CNN
 F 1 "GND" H 3250 3600 50  0000 C CNN
 F 2 "" H 3250 3750 50  0001 C CNN
@@
 	3250 3750 3250 3650
 $Comp
-L GND #PWR21
+L GND #PWR016
 U 1 1 58F1F20B
 P 4600 3550
-F 0 "#PWR21" H 4600 3300 50  0001 C CNN
+F 0 "#PWR016" H 4600 3300 50  0001 C CNN
 F 1 "GND" H 4600 3400 50  0000 C CNN
 F 2 "" H 4600 3550 50  0001 C CNN
@@
 $EndComp
 $Comp
-L +12V #PWR20
+L +12V #PWR017
 U 1 1 58F1F2AA
 P 4600 2400
-F 0 "#PWR20" H 4600 2250 50  0001 C CNN
+F 0 "#PWR017" H 4600 2250 50  0001 C CNN
 F 1 "+12V" H 4600 2540 50  0000 C CNN
 F 2 "" H 4600 2400 50  0001 C CNN
@@
 	4600 2400 4600 2950
 $Comp
-L C C7
+L C C18
 U 1 1 58F1F3A3
 P 4950 2650
-F 0 "C7" H 4975 2750 50  0000 L CNN
+F 0 "C18" H 4975 2750 50  0000 L CNN
 F 1 "0.1" H 4975 2550 50  0000 L CNN
 F 2 "Capacitors_SMD:C_0603" H 4988 2500 50  0001 C CNN
@@
 $EndComp
 $Comp
-L GND #PWR22
+L GND #PWR018
 U 1 1 58F1F415
 P 4950 2800
-F 0 "#PWR22" H 4950 2550 50  0001 C CNN
+F 0 "#PWR018" H 4950 2550 50  0001 C CNN
 F 1 "GND" H 4950 2650 50  0000 C CNN
 F 2 "" H 4950 2800 50  0001 C CNN
@@
 TODO: Low current grounds tie together\nTODO: Place AGND a diode drop lower than this screw term?
 $Comp
-L GND #PWR29
+L GND #PWR019
 U 1 1 58F205D0
 P 6250 4150
-F 0 "#PWR29" H 6250 3900 50  0001 C CNN
+F 0 "#PWR019" H 6250 3900 50  0001 C CNN
 F 1 "GND" H 6250 4000 50  0000 C CNN
 F 2 "" H 6250 4150 50  0001 C CNN
@@
 	6400 5400 6350 5400
 $Comp
-L GND #PWR28
+L GND #PWR020
 U 1 1 58F21660
 P 6050 5700
-F 0 "#PWR28" H 6050 5450 50  0001 C CNN
+F 0 "#PWR020" H 6050 5450 50  0001 C CNN
 F 1 "GND" H 6050 5550 50  0000 C CNN
 F 2 "" H 6050 5700 50  0001 C CNN
@@
 $EndComp
 $Comp
-L +12V #PWR27
+L +12V #PWR021
 U 1 1 58F216B9
 P 6050 4650
-F 0 "#PWR27" H 6050 4500 50  0001 C CNN
+F 0 "#PWR021" H 6050 4500 50  0001 C CNN
 F 1 "+12V" H 6050 4790 50  0000 C CNN
 F 2 "" H 6050 4650 50  0001 C CNN
@@
 	6050 4650 6050 5000
 $Comp
-L C C8
+L C C19
 U 1 1 58F21787
 P 5700 4800
-F 0 "C8" H 5725 4900 50  0000 L CNN
+F 0 "C19" H 5725 4900 50  0000 L CNN
 F 1 "0.1" H 5725 4700 50  0000 L CNN
 F 2 "Capacitors_SMD:C_0603" H 5738 4650 50  0001 C CNN
@@
 Connection ~ 6050 4650
 $Comp
-L GND #PWR25
+L GND #PWR022
 U 1 1 58F218B9
 P 5700 4950
-F 0 "#PWR25" H 5700 4700 50  0001 C CNN
+F 0 "#PWR022" H 5700 4700 50  0001 C CNN
 F 1 "GND" H 5700 4800 50  0000 C CNN
 F 2 "" H 5700 4950 50  0001 C CNN
@@
 	6050 5700 6050 5600
 $Comp
-L GND #PWR26
+L GND #PWR023
 U 1 1 58F24553
 P 5950 5700
-F 0 "#PWR26" H 5950 5450 50  0001 C CNN
+F 0 "#PWR023" H 5950 5450 50  0001 C CNN
 F 1 "GND" H 5950 5550 50  0000 C CNN
 F 2 "" H 5950 5700 50  0001 C CNN
@@
 	5950 5700 5950 5600
 $Comp
-L GND #PWR30
+L GND #PWR024
 U 1 1 58F247EA
 P 6850 6300
-F 0 "#PWR30" H 6850 6050 50  0001 C CNN
+F 0 "#PWR024" H 6850 6050 50  0001 C CNN
 F 1 "GND" H 6850 6150 50  0000 C CNN
 F 2 "" H 6850 6300 50  0001 C CNN
@@
 TODO: zener to restrict +\nTODO: reverse protection
 $Comp
-L CONN_01X02 J1
+L CONN_01X02 J6
 U 1 1 58F251D5
 P 5850 6500
-F 0 "J1" H 5850 6650 50  0000 C CNN
+F 0 "J6" H 5850 6650 50  0000 C CNN
 F 1 "CONN_01X02" V 5950 6500 50  0000 C CNN
 F 2 "Connectors_JST:JST_XH_B02B-XH-A_02x2.50mm_Straight" H 5850 6500 50  0001 C CNN
@@
 	5400 6650 5400 6800
 $Comp
-L +12V #PWR23
+L +12V #PWR025
 U 1 1 58F2577A
 P 5400 6300
-F 0 "#PWR23" H 5400 6150 50  0001 C CNN
+F 0 "#PWR025" H 5400 6150 50  0001 C CNN
 F 1 "+12V" H 5400 6440 50  0000 C CNN
 F 2 "" H 5400 6300 50  0001 C CNN
@@
 $EndComp
 $Comp
-L GND #PWR19
+L GND #PWR026
 U 1 1 58F267F8
 P 3500 7150
-F 0 "#PWR19" H 3500 6900 50  0001 C CNN
+F 0 "#PWR026" H 3500 6900 50  0001 C CNN
 F 1 "GND" H 3500 7000 50  0000 C CNN
 F 2 "" H 3500 7150 50  0001 C CNN
@@
 	4750 7000 4700 7000
 $Comp
-L GND #PWR24
+L GND #PWR027
 U 1 1 58F26CEB
 P 5400 7300
-F 0 "#PWR24" H 5400 7050 50  0001 C CNN
+F 0 "#PWR027" H 5400 7050 50  0001 C CNN
 F 1 "GND" H 5400 7150 50  0000 C CNN
 F 2 "" H 5400 7300 50  0001 C CNN
@@
 	5400 7300 5400 7200
 $Comp
-L +12V #PWR18
+L +12V #PWR028
 U 1 1 58F26E1F
 P 3500 6650
-F 0 "#PWR18" H 3500 6500 50  0001 C CNN
+F 0 "#PWR028" H 3500 6500 50  0001 C CNN
 F 1 "+12V" H 3500 6790 50  0000 C CNN
 F 2 "" H 3500 6650 50  0001 C CNN
@@
 TODO: add resistors to make trim pot\nmore useful
 $Comp
-L R R5
+L R R18
 U 1 1 58F270CD
 P 3050 6850
-F 0 "R5" V 3130 6850 50  0000 C CNN
+F 0 "R18" V 3130 6850 50  0000 C CNN
 F 1 "R" V 3050 6850 50  0000 C CNN
 F 2 "Resistors_SMD:R_0603" V 2980 6850 50  0001 C CNN
@@
 $EndComp
 $Comp
-L GND #PWR16
+L GND #PWR029
 U 1 1 58F2720E
 P 3050 7600
-F 0 "#PWR16" H 3050 7350 50  0001 C CNN
+F 0 "#PWR029" H 3050 7350 50  0001 C CNN
 F 1 "GND" H 3050 7450 50  0000 C CNN
 F 2 "" H 3050 7600 50  0001 C CNN
@@
 	3050 6700 3050 6650
 $Comp
-L +12V #PWR15
+L +12V #PWR030
 U 1 1 58F275E1
 P 3050 6650
-F 0 "#PWR15" H 3050 6500 50  0001 C CNN
+F 0 "#PWR030" H 3050 6500 50  0001 C CNN
 F 1 "+12V" H 3050 6790 50  0000 C CNN
 F 2 "" H 3050 6650 50  0001 C CNN

Commit message: Checkpoint with NHD, 3.3v, and layout
Parts:
- removed D3: D, Diodes_SMD:D_SOD-123, symbol D
- removed J2: Screw_Terminal_1x02, Connectors_Terminal_Blocks:TerminalBlock_Pheonix_MKDS1.5-2pol, symbol Screw_Terminal_1x02
- removed J6: CONN_01X02, Connectors_JST:JST_XH_B02B-XH-A_02x2.50mm_Straight, symbol CONN_01X02
- removed Q1: Q_NMOS_GDS, TO_SOT_Packages_SMD:SOT-23, symbol Q_NMOS_GDS
- removed R18, R19, R20, R23, R24, R25, R26: R, Resistors_SMD:R_0603, symbol R
- removed RV1: POT_TRIM, Potentiometers:Potentiometer_Trimmer_Bourns_3214G, symbol POT_TRIM
- removed TH1: Thermistor_NTC, Connectors_JST:JST_XH_B02B-XH-A_02x2.50mm_Straight, symbol Thermistor_NTC
- removed TP1, TP2, TP3, TP5, TP6, TP7, TP8: TEST, Measurement_Points:Test_Point, symbol TEST
- removed unit 2 of U1
- removed U2: INA128, Housings_SOIC:SOIC-8_3.9x4.9mm_Pitch1.27mm, symbol INA128
- added C2, C3: 0.1, Capacitors_SMD:C_0603, symbol C
- added C?: 4.7n, Capacitors_SMD:C_0603, symbol C
- added D3, D?: D_Schottky, Diodes_SMD:D_SOD-123, symbol D_Schottky
- added J5: Screw_Terminal_1x02, Connectors_Terminal_Blocks:TerminalBlock_Pheonix_MKDS1.5-2pol, symbol Screw_Terminal_1x02
- added R1: 100R, Resistors_SMD:R_0603, symbol R
- added R2: 24K, Resistors_SMD:R_0603, symbol R
- added R3, R? (x2): 10K, Resistors_SMD:R_0603, symbol R
- added R?: 100K, Resistors_SMD:R_0603, symbol R
- C19: value 0.1 -> 4.7n
- Q2, Q3: value Q_NMOS_GDS -> FQP30N06L
- R10: value R -> 4.7K
- R12, R13: value R -> 0R1; footprint Resistors_THT:R_Axial_DIN0516_L15.5mm_D5.0mm_P20.32mm_Horizontal -> Resistors_SMD:R_2512
- R14, R15: value R -> 10K; footprint Resistors_THT:R_Axial_DIN0516_L15.5mm_D5.0mm_P20.32mm_Horizontal -> Resistors_SMD:R_0603
- R7, R8: value R -> 100K
- R9: value R -> 10K
- TP4: footprint Measurement_Points:Test_Point -> Measurement_Points:Measurement_Point_Round-TH_Big
- U1: footprint Housings_SOIC:SOIC-14_3.9x8.7mm_Pitch1.27mm -> (none)
Connections:
- net CHOSEN_VREF: now also U1.12 (+)
- net GND: now also R10.1, R9.2, C2.2, C3.2, C?.2, R3.2, R?.2; no longer R14.2, R15.2, R7.2, U1.11 (V-)
- net at Q2.3 (S), Q3.3 (S), R12.1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: now also U1.3 (+); no longer R14.1, R15.1, R9.1
- net at U1.1, U1.13 (-): now also R2.1; no longer R8.1, R9.2
- net at U1.2 (-): now also R2.2, R3.1; no longer R8.2
- net at R7.1: now also R9.1, U1.10 (+); no longer U1.3 (+)
- net at U1.8: now also R14.2, R15.1; no longer R10.2
- net at U1.9 (-): now also R10.2, R14.1, R8.1
- net at J3.1, Q2.2 (D), Q3.2 (D): now also R?.1
- net at Q2.1 (G), R11.1: now also C3.1
- net at Q3.1 (G), R16.1: now also C2.1
- net +12V: no longer names the net of C18.1, TP4.1, U1.4 (V+)
- net +12V: now also R1.2; no longer C19.1
- new net: J5.1, R7.2
- new net: J5.2, R8.2
- new net: R?.1, R?.1, R?.2
- new net +3V3: D3.1 (K), D?.1 (K), R1.1
- new net LOCAL_SENSE_OUT: C?.1, D?.2 (A), R?.2
- new net REMOTE_SENSE_OUT: C19.1, D3.2 (A), R15.2
Other:
- note added: "Max scale 3v3 = 15A"
- note added: "Notes:\n- Consider FQP50N06L for MOSFET (same form factor, higher dissipation figure)\n- Pay special attention that these grounds are low current"
- note added: "Overvoltage protection\nClamps output to approx 3.6V"
- note added: "Pin 1 positive"
- note added: "RC filter"
- note added: "Reduce short circuit\ncurrent to 33mA"
- note added: "Remote sense (optional)"
- note added: "Shunt is\n2x 0.1 ohm\n= 0.05 ohm equivalent"
- note added: "Textbook divide-by-10-ish\ndifferential amplifier,\n\nOpen input causes approx\n34mV out.\n\nMax current @ 33V = 282uA"
- note added: "Voltage divider"
- note added: "x4.4 amp"
- note removed: "Buffer out of an\nabundance of caution\n(INA is expensive)"
- note removed: "Remote sense"
- note removed: "TODO Rename this for the fact\nit's just scaked voltage across\nthe terminals, and not anything\nto do with current."
- note removed: "TODO diodes vs the main connector as in a PSU?"
- note removed: "TODO: 5V supply for analog"
- note removed: "TODO: Ensure this is 3.3V max (and that we get 30-100C full range)"
- note removed: "TODO: Ensures there is a common ground?\nDoes INA behave without it, or with\na super weak pulldown after the symmetric divider"
- note removed: "TODO: Maybe just series resistor?"
- note removed: "TODO: add resistors to make trim pot\nmore useful"
- note removed: "TODO: damp output a lot"
- note removed: "TODO: look up standard circuit where input may be 36V"
- note removed: "TODO: resistor values for 3.3V = 6.6A,\nhere and shunt."
- note removed: "TODO: simulate and reduce oscillations"
- note removed: "TODO: verify whether paralleled resistor useful for log scale, NYC side"
- note removed: "TODO: zener to restrict +\nTODO: reverse protection"
- moved on the sheet: C18, J3, Q2, Q3, R11, R12, R13, R16, TP4, U1A, U1D
