File: class1.2/resistor_board.kicad_pcb (KiCad board)
At the start: 2 copper layers, 92.7 x 64.1 mm, 14 parts, among them J1 CONN_01X01, J2 CONN_01X01, J3 CONN_01X01, J4 BARREL_JACK, J5 CONN_01X02, M1 ADUINO_MICRO, P1 SYMBOL, P2 SYMBOL

Commit message: Resistor board v0.2
Parts:
- added J6: CONN_01X03, Connectors_Molex:Molex_KK-6410-03_03x2.54mm_Straight, F.Cu at (194.9, 105.4)
- added M2: BuckModule, BuckModule:BuckModule, B.Cu at (153.7, 97.2)
- moved C2 56.0 mm to (194.9, 129.5)
- moved C1 6.35 mm to (130.2, 118.7)
- moved J4 2.54 mm to (121.3, 121.9)
- moved P1 0.63 mm to (127.0, 132.7)
Connections:
- M1 pad 24: Net-(J4-Pad1) -> (no net)
Routing:
- net Net-(J1-Pad1): track 14.8 -> 81.6 mm, vias 0 -> 2
- net Net-(J2-Pad1): track 9.12 -> 58.9 mm, vias 0 -> 2
- net Net-(J4-Pad1): track 21.9 -> 68.3 mm, vias 0 -> 4
- net Net-(J3-Pad1): track 14.5 -> 47.7 mm, vias 0 -> 2
- net +5V: track 161.0 -> 194.1 mm, vias 0 -> 2
- net BUTTON: track 87.1 -> 92.4 mm
- net GND: track 73.1 -> 76.6 mm
- net POT_INPUT: track 48.5 -> 48.1 mm, vias 0 -> 1
Other:
- board text added: "220R"
- board text added: "CC-BY"
- board text added: "Install display last!"
- board text added: "Max 12V"
- board text added: "class1.2 board v0.2"
- board text removed: "CC-A"
- board text removed: "class1.2 board v0.1"

Commit message: Shuffle more footprints.
Parts:
- J1, J2, J3: footprint Connectors-Tim:BANANA_VIA -> Connectors2:BANANA_VIA
- J4: footprint Connectors-Tim:BARREL_JACK -> Connectors2:BARREL_JACK
- moved M2 2.54 mm to (153.7, 99.7)
Routing:
- net Net-(J4-Pad1): track 68.3 -> 66.1 mm
Other:
- board text added: "class1.2 board v0.3-dev"
- board text removed: "class1.2 board v0.2"
Changed lines of the file:
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@@
     (links 40)
     (no_connects 0)
-    (area 107.874999 78.664999 200.735001 142.950001)
+    (area 107.059999 78.639999 200.735001 160.755001)
     (thickness 1.6)
     (drawings 62)
@@
       (xy 8.751927 -1.508911) (xy 9.355248 -1.508911) (xy 9.355248 -0.301782)) (layer F.SilkS) (width 0.01))
   )
-  (module Connectors-Tim:BANANA_VIA (layer F.Cu)
+  (module Connectors2:BANANA_VIA (layer F.Cu)
     (at 139.065 122.555)
     (fp_text reference J1 (at -5.715 0) (layer F.SilkS)
@@
       (net 11 "Net-(J1-Pad1)"))
   )
-  (module Connectors-Tim:BANANA_VIA (layer F.Cu)
+  (module Connectors2:BANANA_VIA (layer F.Cu)
     (at 154.94 122.555)
     (fp_text reference J2 (at -5.715 0) (layer F.SilkS)
@@
       (net 12 "Net-(J2-Pad1)"))
   )
-  (module Connectors-Tim:BANANA_VIA (layer F.Cu)
+  (module Connectors2:BANANA_VIA (layer F.Cu)
     (at 170.815 122.555)
     (fp_text reference J3 (at -5.715 0) (layer F.SilkS)
@@
       (net 16 BUTTON))
   )
-  (module Connectors-Tim:BARREL_JACK (layer B.Cu)
+  (module Connectors2:BARREL_JACK (layer B.Cu)
     (at 121.285 121.92)
     (descr "DC Barrel Jack")
@@
     (pad 3 thru_hole circle (at -3 -4.7) (size 4.2 4.2) (drill 3) (layers *.Cu *.Mask)
       (net 1 GND))
-  )
-  (module BuckModule:BuckModule (layer B.Cu)
-    (at 153.67 97.155 270)
-    (fp_text reference M2 (at 1.27 -6.35 270) (layer B.SilkS)
-      (effects (font (size 1 1) (thickness 0.15)) (justify mirror))
-    )
-    (fp_text value BuckModule (at 0 3.81 270) (layer B.Fab)
-      (effects (font (size 1 1) (thickness 0.15)) (justify mirror))
-    )
-    (fp_line (start -5.08 2.54) (end -5.08 -19.05) (layer B.SilkS) (width 0.15))
-    (fp_line (start 6.35 -19.05) (end 6.35 2.54) (layer B.SilkS) (width 0.15))
-    (fp_text user EN (at 5.08 -2.54 540) (layer B.SilkS)
-      (effects (font (size 1 1) (thickness 0.15)) (justify mirror))
-    )
-    (fp_text user OUT (at 2.54 -2.54 540) (layer B.SilkS)
-      (effects (font (size 1 1) (thickness 0.15)) (justify mirror))
-    )
-    (fp_text user GND (at 0 -2.54 540) (layer B.SilkS)
-      (effects (font (size 1 1) (thickness 0.15)) (justify mirror))
-    )
-    (fp_text user IN (at -2.54 -2.54 540) (layer B.SilkS)
-      (effects (font (size 1 1) (thickness 0.15)) (justify mirror))
-    )
-    (fp_line (start -5.08 2.54) (end 6.35 2.54) (layer B.SilkS) (width 0.15))
-    (fp_line (start 6.35 -19.05) (end -5.08 -19.05) (layer B.SilkS) (width 0.15))
-    (pad 1 thru_hole rect (at -2.54 0 270) (size 1.7 1.7) (drill 1) (layers *.Cu *.Mask)
-      (net 15 "Net-(J4-Pad1)"))
-    (pad 2 thru_hole circle (at 0 0 270) (size 1.7 1.7) (drill 1) (layers *.Cu *.Mask)
-      (net 1 GND))
-    (pad 3 thru_hole circle (at 2.54 0 270) (size 1.7 1.7) (drill 1) (layers *.Cu *.Mask)
-      (net 2 +5V))
-    (pad 4 thru_hole circle (at 5.08 0 270) (size 1.7 1.7) (drill 1) (layers *.Cu *.Mask))
   )
   (module Connectors_Molex:Molex_KK-6410-03_03x2.54mm_Straight (layer F.Cu)
@@
     (pad 24 thru_hole circle (at 7.62 13.97 270) (size 1.7 1.7) (drill 1) (layers *.Cu *.Mask))
   )
+  (module BuckModule:BuckModule (layer B.Cu)
+    (at 153.67 99.695 270)
+    (fp_text reference M2 (at -1.27 -8.255 270) (layer B.SilkS)
+      (effects (font (size 1 1) (thickness 0.15)) (justify mirror))
+    )
+    (fp_text value BuckModule (at -1.27 3.81 270) (layer B.Fab)
+      (effects (font (size 1 1) (thickness 0.15)) (justify mirror))
+    )
+    (fp_line (start -6.985 2.54) (end -6.985 -19.05) (layer B.SilkS) (width 0.15))
+    (fp_line (start 4.445 -19.05) (end 4.445 2.54) (layer B.SilkS) (width 0.15))
+    (fp_text user EN (at -5.08 -2.54 540) (layer B.SilkS)
+      (effects (font (size 1 1) (thickness 0.15)) (justify mirror))
+    )
+    (fp_text user OUT (at 2.54 -2.54 540) (layer B.SilkS)
+      (effects (font (size 1 1) (thickness 0.15)) (justify mirror))
+    )
+    (fp_text user GND (at 0 -2.54 540) (layer B.SilkS)
+      (effects (font (size 1 1) (thickness 0.15)) (justify mirror))
+    )
+    (fp_text user IN (at -2.54 -2.54 540) (layer B.SilkS)
+      (effects (font (size 1 1) (thickness 0.15)) (justify mirror))
+    )
+    (fp_line (start -6.985 2.54) (end 4.445 2.54) (layer B.SilkS) (width 0.15))
+    (fp_line (start 4.445 -19.05) (end -6.985 -19.05) (layer B.SilkS) (width 0.15))
+    (pad 1 thru_hole rect (at -2.54 0 270) (size 1.7 1.7) (drill 1) (layers *.Cu *.Mask)
+      (net 15 "Net-(J4-Pad1)"))
+    (pad 2 thru_hole circle (at 0 0 270) (size 1.7 1.7) (drill 1) (layers *.Cu *.Mask)
+      (net 1 GND))
+    (pad 3 thru_hole circle (at 2.54 0 270) (size 1.7 1.7) (drill 1) (layers *.Cu *.Mask)
+      (net 2 +5V))
+    (pad 4 thru_hole circle (at -5.08 0 270) (size 1.7 1.7) (drill 1) (layers *.Cu *.Mask))
+  )
   (gr_text "Install display last!" (at 161.29 88.265) (layer F.SilkS)
     (effects (font (size 2 2) (thickness 0.3)))
@@
     (effects (font (size 1.5 1.5) (thickness 0.3)))
   )
-  (gr_text "class1.2 board v0.2" (at 127 137.795) (layer F.SilkS)
+  (gr_text "class1.2 board v0.3-dev" (at 127 137.795) (layer F.SilkS)
     (effects (font (size 1.5 1.5) (thickness 0.3)))
   )
@@
   (segment (start 140.97 133.985) (end 142.24 133.985) (width 0.25) (layer B.Cu) (net 2))
   (segment (start 134.62 127.635) (end 140.97 133.985) (width 0.25) (layer B.Cu) (net 2))
-  (segment (start 153.67 99.695) (end 135.89 99.695) (width 0.25) (layer B.Cu) (net 2))
-  (segment (start 131.445 99.695) (end 123.19 99.695) (width 0.25) (layer B.Cu) (net 2))
-  (via (at 131.445 99.695) (size 0.6) (drill 0.4) (layers F.Cu B.Cu) (net 2))
-  (segment (start 135.89 99.695) (end 131.445 99.695) (width 0.25) (layer F.Cu) (net 2))
-  (via (at 135.89 99.695) (size 0.6) (drill 0.4) (layers F.Cu B.Cu) (net 2))
+  (segment (start 153.67 102.235) (end 138.43 102.235) (width 0.25) (layer B.Cu) (net 2) (status 10))
+  (segment (start 134.62 102.235) (end 123.19 102.235) (width 0.25) (layer B.Cu) (net 2))
+  (via (at 134.62 102.235) (size 0.6) (drill 0.4) (layers F.Cu B.Cu) (net 2))
+  (segment (start 138.43 102.235) (end 134.62 102.235) (width 0.25) (layer F.Cu) (net 2))
+  (via (at 138.43 102.235) (size 0.6) (drill 0.4) (layers F.Cu B.Cu) (net 2))
   (segment (start 191.77 98.425) (end 184.15 98.425) (width 0.25) (layer B.Cu) (net 2))
   (segment (start 177.8 92.075) (end 177.8 85.09) (width 0.25) (layer B.Cu) (net 2))
@@
   (segment (start 123.19 83.82) (end 123.19 85.09) (width 0.25) (layer B.Cu) (net 2))
   (segment (start 123.19 104.14) (end 121.92 105.41) (width 0.25) (layer B.Cu) (net 2))
-  (segment (start 123.19 85.09) (end 123.19 99.695) (width 0.25) (layer B.Cu) (net 2))
-  (segment (start 123.19 99.695) (end 123.19 104.14) (width 0.25) (layer B.Cu) (net 2))
+  (segment (start 123.19 85.09) (end 123.19 102.235) (width 0.25) (layer B.Cu) (net 2))
+  (segment (start 123.19 102.235) (end 123.19 104.14) (width 0.25) (layer B.Cu) (net 2))
   (segment (start 124.46 82.55) (end 124.46 81.28) (width 0.25) (layer B.Cu) (net 3))
   (segment (start 124.46 81.28) (end 125.73 80.01) (width 0.25) (layer B.Cu) (net 3))
@@
   (segment (start 150.495 133.985) (end 142.875 133.985) (width 0.25) (layer F.Cu) (net 14))
   (segment (start 153.035 136.525) (end 150.495 133.985) (width 0.25) (layer F.Cu) (net 14))
+  (segment (start 153.67 97.155) (end 155.575 97.155) (width 0.25) (layer B.Cu) (net 15))
+  (segment (start 155.575 97.155) (end 156.845 98.425) (width 0.25) (layer B.Cu) (net 15))
   (segment (start 133.985 129.54) (end 128.905 129.54) (width 0.25) (layer B.Cu) (net 15))
   (segment (start 128.905 129.54) (end 121.285 121.92) (width 0.25) (layer B.Cu) (net 15))
@@
   (via (at 150.495 110.49) (size 0.6) (drill 0.4) (layers F.Cu B.Cu) (net 15))
   (segment (start 150.495 110.49) (end 156.845 104.14) (width 0.25) (layer B.Cu) (net 15))
-  (segment (start 156.845 104.14) (end 156.845 96.52) (width 0.25) (layer B.Cu) (net 15))
-  (segment (start 156.845 96.52) (end 154.94 94.615) (width 0.25) (layer B.Cu) (net 15))
-  (segment (start 154.94 94.615) (end 153.67 94.615) (width 0.25) (layer B.Cu) (net 15))
+  (segment (start 156.845 104.14) (end 156.845 98.425) (width 0.25) (layer B.Cu) (net 15))
   (segment (start 146.685 127) (end 146.685 114.3) (width 0.25) (layer B.Cu) (net 15))
   (via (at 146.685 127) (size 0.6) (drill 0.4) (layers F.Cu B.Cu) (net 15))
